File: rev_a1/nrf52_rev1.kicad_pcb (KiCad board)
At the start: 2 copper layers, 25.4 x 48.3 mm, 27 parts, among them P1 CONN_01X18, P2 CONN_01X18, P3 USB_OTG, U1 nRF52832, U2 CP2102, U3 LT1129CST-3.3, Y1 32K, Y2 32M

Commit message: WIP
Parts:
- added P4: I2C_OLED, Socket_Strips:Socket_Strip_Straight_1x04, F.Cu at (81.3, 27.9)
- P1, P2: moved to F.Cu
- moved Y1 63.2 mm to (116.2, 59.4), turned to 0 degrees
- moved P1 51.0 mm to (27.3, 71.8), turned to 90 degrees
- moved D2 49.3 mm to (29.2, 40.6), turned to 270 degrees
- moved P2 46.4 mm to (27.3, 27.9), turned to 90 degrees
- moved C8 44.0 mm to (104.5, 63.6), turned to 0 degrees
- moved U3 41.7 mm to (36.8, 35.6), turned to 0 degrees
- moved L3 41.1 mm to (102.1, 43.9)
- moved C13 39.2 mm to (102.1, 44.7), turned to 180 degrees
- moved P3 38.8 mm to (27.9, 49.5), turned to 270 degrees
- moved C4 36.6 mm to (104.5, 66.2)
- moved C14 36.4 mm to (106.4, 66.2)
- moved C3 33.7 mm to (103.3, 60.5)
- moved C5 29.6 mm to (104.5, 61.7)
- moved D1 28.6 mm to (44.5, 39.4)
- moved C1 27.1 mm to (96.3, 57.3)
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Connections:
- net 3V3 renamed +3V3
Routing:
- net GND: track 57.1 -> 3.97 mm, vias 3 -> 0
- net Net-(C12-Pad1): track 30.9 -> 0.00 mm
- net P0.20: track 24.5 -> 0.00 mm
- net 5V_IN: track 20.7 -> 0.00 mm
- net P0.21: track 20.7 -> 0.00 mm
- net +5V: track 19.1 -> 0.00 mm
- net SWDCLK: track 17.4 -> 0.00 mm
- net SWDIO: track 14.8 -> 0.00 mm
- net P0.22: track 13.6 -> 0.00 mm
- net P0.23: track 12.4 -> 0.00 mm
- net P0.24: track 12.1 -> 0.00 mm
- net P0.19: track 10.4 -> 0.00 mm
- net P0.08: track 9.35 -> 0.00 mm
- net +3V3: track 10.2 -> 1.58 mm, vias 4 -> 1
- net P0.06: track 8.08 -> 0.00 mm
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Other:
- board size 25.4 x 48.3 mm -> 99.1 x 48.3 mm

Commit message: WIP
Parts:
- C1, C10, C11, C12, C13, C14, C2, C3, C4, C5, C6, C7, C8, C9: footprint RuuviTag:0402_CAP -> RuuviTag:0603_CAP
- L1, L3: footprint RuuviTag:0402_IND -> RuuviTag:0603_IND
- moved Y1 74.3 mm to (44.1, 41.8), turned to 270 degrees
- moved C14 73.9 mm to (37.2, 40.4), turned to 90 degrees
- moved C4 59.6 mm to (47.7, 48.3), turned to 225 degrees
- moved C3 57.3 mm to (50.1, 39.3), turned to 90 degrees
- moved L1 56.4 mm to (49.0, 39.3), turned to 270 degrees
- moved C1 55.8 mm to (42.6, 41.9), turned to 90 degrees
- moved C2 55.2 mm to (45.5, 41.8), turned to 90 degrees
- moved L2 54.8 mm to (48.0, 39.3), turned to 90 degrees
- moved C5 54.6 mm to (54.7, 39.2), turned to 90 degrees
- moved C6 54.2 mm to (47.0, 39.3), turned to 90 degrees
- moved C7 53.8 mm to (46.0, 39.3), turned to 90 degrees
- moved C9 50.5 mm to (58.1, 45.1), turned to 270 degrees
- moved C8 49.0 mm to (59.2, 45.1), turned to 270 degrees
- moved L3 43.6 mm to (58.6, 47.9)
- moved C13 41.9 mm to (60.3, 47.2), turned to 90 degrees
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Connections:
- P2 pad 1: P0.31 -> GND
- P2 pad 10: P0.22 -> P0.26
- P2 pad 11: SWDIO -> P0.25
- P2 pad 12: SWDCLK -> P0.24
- P2 pad 13: P0.21 -> P0.23
- P2 pad 14: P0.20 -> P0.22
- P2 pad 15: +3V3 -> SWDIO
- P2 pad 16: GND -> SWDCLK
- P2 pad 17: 5V_IN -> P0.21
- P2 pad 18: GND -> P0.20
- P2 pad 2: P0.30 -> 5V_IN
- P2 pad 3: P0.29 -> GND
- P2 pad 4: P0.28 -> +3V3
- P2 pad 5: P0.27 -> P0.31
- P2 pad 6: P0.26 -> P0.30
- P2 pad 7: P0.25 -> P0.29
- P2 pad 8: P0.24 -> P0.28
- P2 pad 9: P0.23 -> P0.27
Routing:
- net 5V_IN: track 0.00 -> 24.7 mm
- net GND: track 3.97 -> 27.4 mm
- net +3V3: track 1.58 -> 21.7 mm, vias 1 -> 6
- net /ANTENNA: track 0.00 -> 16.9 mm
- net +5V: track 0.00 -> 13.6 mm
- net USB_D+: track 0.00 -> 11.5 mm, vias 0 -> 2
- net USB_D-: track 0.00 -> 10.3 mm, vias 0 -> 2
- net XL1: track 0.00 -> 7.63 mm
- net XL2: track 0.00 -> 6.85 mm
- net Net-(C8-Pad1): track 0.00 -> 5.95 mm
- net Net-(C12-Pad1): track 0.00 -> 5.43 mm
- net P0.25: track 0.00 -> 4.99 mm
- net P0.26: track 0.00 -> 4.73 mm
- net P0.27: track 0.00 -> 4.59 mm
- net Net-(D1-Pad2): track 0.00 -> 4.57 mm
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Other:
- net class Power added: clearance 0.0762, trace_width 0.4064, via_dia 0.6, via_drill 0.3

Commit message: Wiiip
Parts:
- moved P4 43.2 mm to (74.7, 70.6)
- moved P1 12.7 mm to (27.9, 71.1)
- moved U2 11.1 mm to (31.0, 59.4)
- moved D1 8.18 mm to (35.6, 41.7)
- moved C11 5.80 mm to (55.0, 45.1)
- moved C13 5.80 mm to (58.0, 52.5)
- moved C2 5.80 mm to (43.2, 47.2)
- moved C3 5.80 mm to (47.8, 44.6)
- moved C5 5.80 mm to (52.5, 44.6)
- moved C6 5.80 mm to (44.7, 44.6)
- moved C7 5.80 mm to (43.7, 44.6)
- moved L1 5.80 mm to (46.8, 44.6)
- moved L2 5.80 mm to (45.7, 44.6)
- moved L3 5.80 mm to (56.4, 53.2)
- moved U1 5.80 mm to (49.4, 49.5)
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Routing:
- net +5V: track 13.6 -> 27.7 mm, vias 0 -> 2
- net Net-(D1-Pad2): track 4.57 -> 9.35 mm
- net +3V3: track 21.7 -> 18.6 mm, vias 6 -> 5
- net USB_D+: track 11.5 -> 8.79 mm, vias 2 -> 0
- net 5V_IN: track 24.7 -> 26.4 mm

Commit message: Wörk wörk
Parts:
- removed P4: I2C_OLED, Socket_Strips:Socket_Strip_Straight_1x04
Routing:
- net GND: track 27.4 -> 74.5 mm, vias 0 -> 3
- net P0.02: track 0.00 -> 35.5 mm
- net P0.05: track 0.00 -> 34.4 mm, vias 0 -> 2
- net P0.03: track 0.00 -> 33.3 mm
- net P0.08: track 0.00 -> 32.3 mm, vias 0 -> 2
- net P0.19: track 0.00 -> 31.8 mm
- net P0.06: track 0.00 -> 31.6 mm, vias 0 -> 2
- net P0.07: track 0.00 -> 30.8 mm, vias 0 -> 2
- net P0.04: track 0.00 -> 30.5 mm
- net P0.18: track 0.00 -> 28.8 mm
- net P0.17: track 0.00 -> 27.8 mm
- net P0.16: track 0.00 -> 26.0 mm
- net P0.31: track 3.87 -> 28.0 mm
- net P0.15: track 0.00 -> 22.7 mm
- net P0.30: track 4.19 -> 25.9 mm
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Other:
- board size 99.1 x 48.3 mm -> 48.3 x 48.3 mm
- net class Power_3v3 added: clearance 0.0762, trace_width 0.3048, via_dia 0.6, via_drill 0.3

Commit message: wipwipwip
Parts:
- added C15: 4u7, RuuviTag:0603_CAP, F.Cu at (26.9, 56.4)
- added C16: 4u7, RuuviTag:0603_CAP, F.Cu at (32.8, 54.9)
- added C17: 100n, RuuviTag:0603_CAP, F.Cu at (33.8, 54.9)
- added R1: 4k7, RuuviTag:0603_RES, F.Cu at (29.2, 64.1)
Routing:
- net +3V3: track 26.5 -> 35.4 mm, vias 6 -> 8
- net Net-(R1-Pad1): track 0.00 -> 7.42 mm
- net GND: track 74.5 -> 78.6 mm
- net +5V: track 27.7 -> 29.6 mm

Commit message: wörk wörk
Routing:
- net P0.24: track 0.00 -> 77.1 mm
- net P0.23: track 0.00 -> 76.1 mm
- net P0.22: track 0.32 -> 75.6 mm
- net SWDCLK: track 4.40 -> 73.1 mm
- net P0.20: track 4.16 -> 72.6 mm
- net SWDIO: track 7.74 -> 75.6 mm
- net P0.21: track 4.46 -> 71.8 mm
- net GND: track 78.6 -> 71.7 mm
- net P0.12: track 18.8 -> 19.8 mm

Commit message: wip
Parts:
- moved Y2 2.23 mm to (56.1, 45.0), turned to 180 degrees
- moved C10 2.08 mm to (56.4, 47.0)
- moved C12 1.52 mm to (56.4, 50.6)
- moved C13 1.52 mm to (58.0, 51.0)
- moved C8 1.52 mm to (56.9, 48.9)
- moved C9 1.52 mm to (55.8, 48.9)
- moved L3 1.52 mm to (56.4, 51.7)
- moved C11 0.90 mm to (54.1, 45.0), turned to 270 degrees
- moved C5 0.43 mm to (52.6, 45.0)
Routing:
- net P0.02: track 35.5 -> 0.00 mm
- net P0.03: track 33.2 -> 1.02 mm
- net P0.04: track 30.5 -> 0.00 mm
- net P0.31: track 28.0 -> 0.00 mm
- net P0.30: track 25.9 -> 0.00 mm
- net P0.29: track 23.9 -> 0.00 mm
- net P0.28: track 21.8 -> 0.00 mm
- net P0.27: track 19.8 -> 0.00 mm
- net P0.25: track 19.4 -> 0.00 mm
- net P0.26: track 18.9 -> 0.57 mm
- net P0.11: track 19.5 -> 2.66 mm
- net P0.05: track 34.4 -> 18.3 mm
- net P0.24: track 77.1 -> 61.4 mm
- net P0.22: track 75.6 -> 60.1 mm
- net P0.23: track 76.1 -> 60.7 mm
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
Commit message: wip
Parts:
- moved C15 19.1 mm to (40.8, 43.2), turned to 180 degrees
- moved R1 19.0 mm to (35.4, 46.2), turned to 90 degrees
- moved C16 13.2 mm to (40.8, 44.4), turned to 180 degrees
- moved U2 11.9 mm to (38.2, 50.0), turned to 225 degrees
- moved C17 11.6 mm to (40.8, 45.6), turned to 180 degrees
- moved C1 10.1 mm to (44.5, 38.0), turned to 0 degrees
- moved C7 10.0 mm to (42.4, 34.7)
- moved C6 10.00 mm to (43.6, 34.7)
- moved L2 9.99 mm to (44.7, 34.7)
- moved L1 9.96 mm to (46.0, 34.7)
- moved C3 9.95 mm to (47.1, 34.7)
- moved Y1 9.23 mm to (46.5, 39.2)
- moved C12 8.84 mm to (60.6, 42.9)
- moved L3 8.69 mm to (60.6, 44.1)
- moved C9 8.65 mm to (59.3, 41.0), turned to 0 degrees
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Routing:
- net P0.24: track 61.4 -> 0.00 mm
- net P0.23: track 60.7 -> 0.00 mm
- net P0.22: track 60.1 -> 0.00 mm
- net P0.20: track 59.3 -> 0.00 mm
- net SWDCLK: track 59.3 -> 0.10 mm
- net SWDIO: track 60.4 -> 1.65 mm
- net P0.21: track 58.6 -> 0.00 mm
- net GND: track 69.4 -> 100.7 mm, vias 3 -> 4
- net P0.31: track 0.00 -> 23.2 mm
- net P0.08: track 21.6 -> 0.00 mm, vias 2 -> 0
- net P0.30: track 0.00 -> 20.3 mm
- net P0.05: track 18.3 -> 0.00 mm, vias 2 -> 0
- net P0.06: track 18.3 -> 0.00 mm, vias 2 -> 0
- net P0.19: track 18.3 -> 0.00 mm
- net P0.29: track 0.00 -> 18.2 mm
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