File: rev_a1/nrf52_rev1.kicad_pcb (KiCad board)
At the start: 2 copper layers, 48.3 x 48.3 mm, 31 parts, among them P1 CONN_01X18, P2 CONN_01X18, P3 USB_OTG, U1 nRF52832, U2 CP2102, U3 LT1129CST-3.3, Y1 32K, Y2 32M

Commit message: wip
Connections:
- U2 pad 23: P0.05 -> P0.08
- U2 pad 26: P0.08 -> P0.05
Routing:
- net P0.05: track 0.00 -> 60.0 mm, vias 0 -> 2
- net P0.06: track 0.00 -> 55.2 mm, vias 0 -> 2
- net P0.07: track 0.00 -> 51.4 mm, vias 0 -> 2
- net P0.08: track 0.00 -> 50.8 mm, vias 0 -> 2
- net P0.02: track 0.00 -> 46.4 mm
- net P0.03: track 0.00 -> 44.8 mm
- net P0.04: track 0.00 -> 41.2 mm
- net +3V3: track 25.0 -> 27.5 mm, vias 5 -> 7
- net GND: track 100.7 -> 98.8 mm

Commit message: wip
Parts:
- moved C10 10.6 mm to (70.0, 38.9)
- moved C11 10.6 mm to (67.7, 36.9)
- moved C12 10.6 mm to (71.2, 42.1)
- moved C3 10.6 mm to (57.7, 33.8)
- moved C4 10.6 mm to (60.0, 46.3)
- moved C5 10.6 mm to (66.1, 36.9)
- moved C6 10.6 mm to (54.2, 33.8)
- moved C7 10.6 mm to (53.0, 33.8)
- moved C9 10.6 mm to (70.0, 40.2)
- moved L1 10.6 mm to (56.6, 33.8)
- moved L2 10.6 mm to (55.3, 33.8)
- moved U1 10.6 mm to (63.0, 41.4)
- moved Y1 10.6 mm to (57.1, 38.4)
- moved C1 10.6 mm to (55.1, 37.1)
- moved C13 10.6 mm to (71.2, 44.4)
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Connections:
- P1 pad 1: P0.02 -> P0.11
- P1 pad 10: P0.13 -> P0.20
- P1 pad 11: P0.14 -> P0.21
- P1 pad 12: P0.15 -> SWDCLK
- P1 pad 13: P0.16 -> SWDIO
- P1 pad 14: P0.17 -> P0.22
- P1 pad 15: P0.18 -> P0.23
- P1 pad 16: P0.19 -> P0.24
- P1 pad 2: P0.03 -> P0.12
- P1 pad 3: P0.04 -> P0.13
- P1 pad 4: P0.05 -> P0.14
- P1 pad 5: P0.06 -> P0.15
- P1 pad 6: P0.07 -> P0.16
- P1 pad 7: P0.08 -> P0.17
- P1 pad 8: P0.11 -> P0.18
- P1 pad 9: P0.12 -> P0.19
- P2 pad 10: P0.26 -> P0.03
- P2 pad 11: P0.25 -> P0.02
- P2 pad 12: P0.24 -> P0.31
- P2 pad 13: P0.23 -> P0.30
- P2 pad 14: P0.22 -> P0.29
- P2 pad 15: SWDIO -> P0.28
- P2 pad 16: SWDCLK -> P0.27
- P2 pad 17: P0.21 -> P0.26
- P2 pad 18: P0.20 -> P0.25
- P2 pad 5: P0.31 -> P0.08
- P2 pad 6: P0.30 -> P0.07
- P2 pad 7: P0.29 -> P0.06
- P2 pad 8: P0.28 -> P0.05
- P2 pad 9: P0.27 -> P0.04
Routing:
- net P0.05: track 60.0 -> 26.4 mm, vias 2 -> 0
- net P0.06: track 55.2 -> 29.2 mm, vias 2 -> 0
- net P0.02: track 46.4 -> 20.5 mm
- net P0.03: track 44.8 -> 21.0 mm
- net P0.07: track 51.4 -> 31.9 mm, vias 2 -> 0
- net P0.04: track 41.2 -> 23.5 mm
- net P0.08: track 50.8 -> 35.4 mm, vias 2 -> 0
- net P0.31: track 23.2 -> 17.0 mm
- net P0.24: track 0.00 -> 6.27 mm
- net P0.30: track 20.3 -> 14.6 mm
- net P0.29: track 18.2 -> 12.7 mm
- net P0.23: track 0.00 -> 5.39 mm
- net (no net): track 0.00 -> 5.21 mm, vias 0 -> 2
- net P0.22: track 0.00 -> 4.42 mm
- net P0.28: track 16.4 -> 12.5 mm
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
Commit message: wip
Parts:
- moved R1 1.49 mm to (33.9, 46.1)
- moved C14 1.15 mm to (32.9, 46.1)
Routing:
- net P0.08: track 35.4 -> 64.8 mm, vias 0 -> 2
- net P0.05: track 26.4 -> 55.4 mm, vias 0 -> 2
- net P0.06: track 29.2 -> 56.9 mm, vias 0 -> 2
- net P0.07: track 31.9 -> 59.3 mm, vias 0 -> 2
- net +5V: track 20.8 -> 6.90 mm
- net USB_D+: track 15.5 -> 27.3 mm, vias 2 -> 0
- net USB_D-: track 13.7 -> 23.4 mm, vias 2 -> 0
- net P0.24: track 6.27 -> 0.00 mm
- net GND: track 98.8 -> 92.8 mm
- net P0.23: track 5.39 -> 0.00 mm
- net (no net): track 5.21 -> 0.00 mm, vias 2 -> 0
- net P0.22: track 4.42 -> 0.00 mm
- net Net-(R1-Pad1): track 2.10 -> 3.71 mm, vias 0 -> 2

Commit message: wip
Routing:
- net P0.11: track 0.00 -> 60.9 mm
- net P0.24: track 0.00 -> 32.5 mm
- net GND: track 92.8 -> 120.1 mm, vias 4 -> 10
- net +5V: track 6.90 -> 22.5 mm, vias 0 -> 3
- net USB_D+: track 27.3 -> 26.2 mm
- net USB_D-: track 23.4 -> 24.1 mm

Commit message: Made the design great again
Parts:
- moved U2 14.5 mm to (42.8, 36.3), turned to 0 degrees
- moved R1 10.7 mm to (43.1, 40.5), turned to 0 degrees
- moved C15 9.54 mm to (32.6, 48.1), turned to 90 degrees
- moved C16 7.47 mm to (37.2, 37.8), turned to 0 degrees
- moved C17 7.41 mm to (37.2, 39.1), turned to 0 degrees
- moved C11 5.21 mm to (62.5, 36.9)
- moved C4 5.21 mm to (54.8, 46.3)
- moved C5 5.21 mm to (60.9, 36.9)
- moved U1 5.21 mm to (57.8, 41.4)
- moved C10 5.21 mm to (64.7, 38.9)
- moved C12 5.21 mm to (66.0, 42.1)
- moved C13 5.21 mm to (66.0, 44.4)
- moved C8 5.21 mm to (64.3, 43.8)
- moved C9 5.21 mm to (64.7, 40.2)
- moved L3 5.21 mm to (66.0, 43.2)
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Connections:
- U2 pad 23: P0.08 -> P0.05
- U2 pad 24: P0.07 -> P0.06
- U2 pad 25: P0.06 -> P0.07
- U2 pad 26: P0.05 -> P0.08
Routing:
- net P0.11: track 60.9 -> 0.00 mm
- net P0.24: track 32.5 -> 0.00 mm
- net P0.08: track 64.8 -> 32.5 mm, vias 2 -> 0
- net P0.05: track 55.4 -> 26.2 mm
- net P0.06: track 56.9 -> 28.3 mm
- net P0.07: track 59.3 -> 32.5 mm
- net GND: track 120.1 -> 109.0 mm, vias 10 -> 7
- net 5V_IN: track 25.0 -> 33.0 mm, vias 0 -> 2
- net P0.31: track 17.0 -> 11.6 mm
- net P0.27: track 11.3 -> 16.0 mm
- net Net-(D1-Pad2): track 9.35 -> 4.84 mm
- net P0.25: track 15.8 -> 20.2 mm
- net P0.26: track 14.0 -> 18.1 mm
- net +5V: track 22.5 -> 26.3 mm, vias 3 -> 2
- net P0.30: track 14.6 -> 10.8 mm
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Other:
- net class Default: clearance 0.0762 -> 0.1524
- rule trace_clearance: 0.0762 -> 0.1524

Commit message: woo
Parts:
- moved C8 2.78 mm to (66.1, 41.7), turned to 0 degrees
- moved C12 0.62 mm to (66.1, 42.7)
- moved L3 0.46 mm to (66.1, 43.7)
- moved C13 0.34 mm to (66.1, 44.7)
Routing:
- net GND: track 109.0 -> 115.2 mm, vias 7 -> 8
- net Net-(C8-Pad1): track 5.59 -> 7.09 mm

Commit message: Added logo etc
Parts:
- added G***: LOGO, xil_assets:logo_inv, B.Cu at (50.8, 49.5)
Routing:
- net GND: track 115.2 -> 117.2 mm
- net Net-(L1-Pad1): track 1.27 -> 2.48 mm
- net Net-(C3-Pad1): track 6.13 -> 7.28 mm
- net Net-(C7-Pad1): track 6.85 -> 6.18 mm

Commit message: Almost done
Parts:
- removed G***: LOGO, xil_assets:logo_inv
- added ?: , xil_assets:ti-an043-antenna-mask, F.Cu at (67.3, 42.2)
- added P4: ANTENNA_2_4GHZ, xil_assets:ti-an043-antenna, F.Cu at (67.3, 42.2)
- moved C12 0.51 mm to (65.6, 42.7)
- moved C13 0.51 mm to (65.6, 44.7)
- moved C8 0.51 mm to (65.6, 41.7)
- moved L3 0.51 mm to (65.6, 43.7)
Routing:
- net P0.11: track 0.00 -> 56.8 mm
- net P0.12: track 0.00 -> 54.9 mm
- net P0.13: track 0.00 -> 52.6 mm
- net P0.14: track 0.00 -> 50.4 mm
- net P0.15: track 0.00 -> 48.3 mm
- net P0.16: track 0.00 -> 46.2 mm
- net P0.17: track 0.00 -> 44.1 mm
- net P0.18: track 0.00 -> 42.0 mm
- net P0.19: track 0.00 -> 39.9 mm
- net P0.20: track 0.00 -> 37.7 mm
- net P0.21: track 0.00 -> 35.6 mm
- net SWDCLK: track 0.10 -> 34.2 mm
- net SWDIO: track 0.00 -> 32.8 mm
- net P0.22: track 0.00 -> 32.8 mm
- net P0.23: track 0.00 -> 32.5 mm
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Other:
- net class Default: clearance 0.1524 -> 0.0762
- rule trace_clearance: 0.1524 -> 0.0762
