File: rev_a1/nrf52_rev1.kicad_pcb (KiCad board)
At the start: 2 copper layers, 48.3 x 48.3 mm, 37 parts, among them P1 CONN_01X18, P2 CONN_01X18, P3 USB_OTG, P4 ANTENNA_2_4GHZ, U1 nRF52832, U2 CP2102, U3 LT1129CST-3.3, Y1 32K, Y2 32M

Commit message: uhh, hope this works
Parts:
- added JP1: Jumper_NO_Small, xil_assets:SolderBridgeLarge, B.Cu at (43.6, 30.3)
- added JP2: Jumper_NO_Small, xil_assets:SolderBridgeLarge, B.Cu at (46.1, 30.3)
- moved C7 1.78 mm to (50.4, 33.8)
- moved C6 1.40 mm to (51.9, 33.8)
- moved R1 1.40 mm to (33.8, 37.1)
- moved L2 1.02 mm to (53.5, 33.8)
- moved C13 1.02 mm to (65.5, 45.7)
- moved C17 1.02 mm to (35.3, 37.1)
- moved L3 0.76 mm to (65.5, 44.5)
- moved C16 0.76 mm to (36.8, 37.1)
- moved L1 0.70 mm to (55.0, 33.8)
- moved C12 0.51 mm to (65.5, 43.2)
- moved ? 0.50 mm to (67.3, 42.7)
- moved P4 0.50 mm to (67.3, 42.7)
- moved C14 0.38 mm to (38.4, 37.1)
- moved C3 0.32 mm to (56.5, 33.8)
- moved C8 0.26 mm to (65.5, 41.9)
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Connections:
- net USB_D+ renamed /CP2102/USB_D+
- net USB_D- renamed /CP2102/USB_D-
- U2 pad 23: P0.05 -> /CP2102/UART_CTS
- U2 pad 24: P0.06 -> /CP2102/UART_RTS
Routing:
- net /CP2102/UART_CTS: track 0.00 -> 4.42 mm, vias 0 -> 1
- net P0.05: track 25.5 -> 21.5 mm, vias 2 -> 1
- net +3V3: track 29.8 -> 32.7 mm
- net /CP2102/UART_RTS: track 0.00 -> 2.89 mm, vias 0 -> 1
- net GND: track 170.6 -> 167.8 mm
- net P0.06: track 26.9 -> 24.2 mm, vias 2 -> 1
- net Net-(C7-Pad1): track 6.18 -> 7.88 mm
- net Net-(R1-Pad1): track 7.87 -> 9.43 mm
- net Net-(L1-Pad1): track 2.48 -> 1.52 mm
- net XC1: track 9.09 -> 9.62 mm
Other:
- outline, holes or cut-outs redrawn

Commit message: foo
Parts:
- added G***: LOGO, xil_assets:nfc_30x18_w05mm_s06mm_sm, F.Cu at (41.0, 56.0)
- added P5: ANTENNA_NFC, xil_assets:nfc_30x18_w05mm_s06mm, F.Cu at (41.1, 56.0)
Routing:
- net NFC2: track 5.75 -> 19.2 mm, vias 0 -> 2
- net (no net): track 12.0 -> 0.17 mm, vias 2 -> 0
- net NFC1: track 6.71 -> 13.2 mm
- net GND: track 167.8 -> 173.6 mm, vias 12 -> 14

Commit message: soon going gold
Parts:
- removed the G*** at (41.0, 56.0)
- added G***: LOGO, xil_assets:logo_23x19mm, F.Cu at (41.4, 55.7)

Commit message: changed diode connections
Parts:
- added G***: LOGO, xil_assets:logo_26x20mm, B.Cu at (50.0, 48.3)
- D1, D2: value D_Schottky -> D; footprint Diodes_SMD:SOD-123 -> Diodes_SMD:SOD-323
- moved D2 0.56 mm to (36.6, 34.0)
- moved D1 0.51 mm to (36.6, 32.0)
- moved C15 0.20 mm to (35.4, 40.7)
Connections:
- D2 pad 1: +3V3 -> +5V
- D2 pad 2: Net-(D2-Pad2) -> +3V3
- U3 pad 3: Net-(D2-Pad2) -> +3V3
Routing:
- net Net-(D2-Pad2): track 15.8 -> 0.00 mm, vias 2 -> 0
- net GND: track 173.6 -> 180.4 mm
- net +5V: track 16.6 -> 18.7 mm
- net +3V3: track 33.2 -> 31.6 mm
- net 5V_IN: track 13.6 -> 14.8 mm
- net /CP2102/USB_D+: track 21.2 -> 21.8 mm
Other:
- board text added: "NRF52832 NFC+BT DESIGNED BY KBECKMANN REV A1 2016-06"
