File: rev_a1/nrf52_rev1.sch (KiCad schematic (older format))
At the start: 31 parts, among them P1 CONN_01X18, P2 CONN_01X18, P3 USB_OTG, U1 nRF52832, U2 CP2102, U3 LT1129CST-3.3, Y1 32K, Y2 32M

Commit message: Made the design great again
Connections:
- net P0.05: now also U2.23 (CTS); no longer U2.26 (TXD)
- net P0.06: now also U2.24 (RTS); no longer U2.25 (RXD)
- net P0.07: now also U2.25 (RXD); no longer U2.24 (RTS)
- net P0.08: now also U2.26 (TXD); no longer U2.23 (CTS)
Changed lines of the file:
@@
 Text GLabel 5050 6650 2    47   Input ~ 0
 UART_CTS
+Text GLabel 2500 2900 0    47   Input ~ 0
+UART_TXD
+Text GLabel 2500 2800 0    47   Input ~ 0
+UART_RXD
+Text GLabel 2500 2700 0    47   Input ~ 0
+UART_RTS
 Text GLabel 2500 2600 0    47   Input ~ 0
-UART_TXD
-Text GLabel 2500 2700 0    47   Input ~ 0
-UART_RXD
-Text GLabel 2500 2800 0    47   Input ~ 0
-UART_RTS
-Text GLabel 2500 2900 0    47   Input ~ 0
 UART_CTS
 Text GLabel 1150 6650 2    47   Input ~ 0

Commit message: Added logo etc
Parts:
- added P?: CONN_01X01, symbol CONN_01X01
Changed lines of the file:
@@
 LIBS:tmp007
 LIBS:uvis25
+LIBS:tom_kicad
 LIBS:nrf52_rev1-cache
 EELAYER 25 0
@@
 Wire Wire Line
 	4250 5250 4250 5650
+$Comp
+L CONN_01X01 P?
+U 1 1 5762FAFE
+P 8650 1650
+F 0 "P?" H 8728 1691 50  0000 L CNN
+F 1 "CONN_01X01" H 8728 1600 50  0000 L CNN
+F 2 "" H 8650 1650 50  0000 C CNN
+F 3 "" H 8650 1650 50  0000 C CNN
+	1    8650 1650
+	1    0    0    -1
+$EndComp
 $EndSCHEMATC

Commit message: Almost done
Parts:
- removed P?: CONN_01X01, symbol CONN_01X01
- added P4: ANTENNA_2_4GHZ, xil_assets:ti-an043-antenna, symbol CONN_02X01
Connections:
- net ANTENNA: now also P4.1 (P1)
- net GND: now also P4.2 (P2)
Changed lines of the file:
@@
 $EndDescr
 $Comp
-L GND #PWR01
+L GND #PWR28
 U 1 1 57587EFC
 P 6300 1300
-F 0 "#PWR01" H 6300 1050 50  0001 C CNN
+F 0 "#PWR28" H 6300 1050 50  0001 C CNN
 F 1 "GND" H 6300 1150 50  0000 C CNN
 F 2 "" H 6300 1300 50  0000 C CNN
@@
 $EndComp
 $Comp
-L GND #PWR02
+L GND #PWR9
 U 1 1 57588077
 P 2450 1000
-F 0 "#PWR02" H 2450 750 50  0001 C CNN
+F 0 "#PWR9" H 2450 750 50  0001 C CNN
 F 1 "GND" V 2449 812 50  0000 C CNN
 F 2 "" H 2450 1000 50  0000 C CNN
@@
 $EndComp
 $Comp
-L GND #PWR03
+L GND #PWR8
 U 1 1 57588655
 P 2450 900
-F 0 "#PWR03" H 2450 650 50  0001 C CNN
+F 0 "#PWR8" H 2450 650 50  0001 C CNN
 F 1 "GND" V 2449 712 50  0000 C CNN
 F 2 "" H 2450 900 50  0000 C CNN
@@
 $EndComp
 $Comp
-L GND #PWR04
+L GND #PWR7
 U 1 1 5758866C
 P 2450 800
-F 0 "#PWR04" H 2450 550 50  0001 C CNN
+F 0 "#PWR7" H 2450 550 50  0001 C CNN
 F 1 "GND" V 2449 612 50  0000 C CNN
 F 2 "" H 2450 800 50  0000 C CNN
@@
 $EndComp
 $Comp
-L GND #PWR05
+L GND #PWR12
 U 1 1 575887A0
 P 2450 1400
-F 0 "#PWR05" H 2450 1150 50  0001 C CNN
+F 0 "#PWR12" H 2450 1150 50  0001 C CNN
 F 1 "GND" V 2449 1212 50  0000 C CNN
 F 2 "" H 2450 1400 50  0000 C CNN
@@
 $EndComp
 $Comp
-L GND #PWR06
+L GND #PWR11
 U 1 1 575887B8
 P 2450 1300
-F 0 "#PWR06" H 2450 1050 50  0001 C CNN
+F 0 "#PWR11" H 2450 1050 50  0001 C CNN
 F 1 "GND" V 2449 1112 50  0000 C CNN
 F 2 "" H 2450 1300 50  0000 C CNN
@@
 $EndComp
 $Comp
-L GND #PWR07
+L GND #PWR10
 U 1 1 575887BE
 P 2450 1200
-F 0 "#PWR07" H 2450 950 50  0001 C CNN
+F 0 "#PWR10" H 2450 950 50  0001 C CNN
 F 1 "GND" V 2449 1012 50  0000 C CNN
 F 2 "" H 2450 1200 50  0000 C CNN
@@
 $EndComp
 $Comp
-L GND #PWR08
+L GND #PWR13
 U 1 1 57589680
 P 2450 1700
-F 0 "#PWR08" H 2450 1450 50  0001 C CNN
+F 0 "#PWR13" H 2450 1450 50  0001 C CNN
 F 1 "GND" V 2449 1512 50  0000 C CNN
 F 2 "" H 2450 1700 50  0000 C CNN
@@
 $EndComp
 $Comp
-L GND #PWR09
+L GND #PWR15
 U 1 1 57589C6C
 P 3050 3500
-F 0 "#PWR09" H 3050 3250 50  0001 C CNN
+F 0 "#PWR15" H 3050 3250 50  0001 C CNN
 F 1 "GND" V 3049 3312 50  0000 C CNN
 F 2 "" H 3050 3500 50  0000 C CNN
@@
 $EndComp
 $Comp
-L GND #PWR010
+L GND #PWR18
 U 1 1 57589C95
 P 3650 4000
-F 0 "#PWR010" H 3650 3750 50  0001 C CNN
+F 0 "#PWR18" H 3650 3750 50  0001 C CNN
 F 1 "GND" V 3649 3812 50  0000 C CNN
 F 2 "" H 3650 4000 50  0000 C CNN
@@
 $EndComp
 $Comp
-L GND #PWR011
+L GND #PWR19
 U 1 1 57589CBE
 P 3650 4100
-F 0 "#PWR011" H 3650 3850 50  0001 C CNN
+F 0 "#PWR19" H 3650 3850 50  0001 C CNN
 F 1 "GND" V 3649 3912 50  0000 C CNN
 F 2 "" H 3650 4100 50  0000 C CNN
@@
 $EndComp
 $Comp
-L GND #PWR012
+L GND #PWR26
 U 1 1 5758A08F
 P 5200 4100
-F 0 "#PWR012" H 5200 3850 50  0001 C CNN
+F 0 "#PWR26" H 5200 3850 50  0001 C CNN
 F 1 "GND" V 5199 3912 50  0000 C CNN
 F 2 "" H 5200 4100 50  0000 C CNN
@@
 $EndComp
 $Comp
-L GND #PWR013
+L GND #PWR25
 U 1 1 5758A0C1
 P 5200 4000
-F 0 "#PWR013" H 5200 3750 50  0001 C CNN
+F 0 "#PWR25" H 5200 3750 50  0001 C CNN
 F 1 "GND" V 5199 3812 50  0000 C CNN
 F 2 "" H 5200 4000 50  0000 C CNN
@@
 $EndComp
 $Comp
-L GND #PWR014
+L GND #PWR5
 U 1 1 5758E3CC
 P 1650 5450
-F 0 "#PWR014" H 1650 5200 50  0001 C CNN
+F 0 "#PWR5" H 1650 5200 50  0001 C CNN
 F 1 "GND" H 1650 5300 50  0000 C CNN
 F 2 "" H 1650 5450 50  0000 C CNN
@@
 $EndComp
 $Comp
-L PWR_FLAG #FLG015
+L PWR_FLAG #FLG2
 U 1 1 5758E406
 P 2050 5400
-F 0 "#FLG015" H 2050 5495 50  0001 C CNN
+F 0 "#FLG2" H 2050 5495 50  0001 C CNN
 F 1 "PWR_FLAG" H 2050 5580 50  0000 C CNN
 F 2 "" H 2050 5400 50  0000 C CNN
@@
 $EndComp
 $Comp
-L PWR_FLAG #FLG016
+L PWR_FLAG #FLG3
 U 1 1 5758E498
 P 2550 5100
-F 0 "#FLG016" H 2550 5195 50  0001 C CNN
+F 0 "#FLG3" H 2550 5195 50  0001 C CNN
 F 1 "PWR_FLAG" H 2550 5280 50  0000 C CNN
 F 2 "" H 2550 5100 50  0000 C CNN
@@
 $EndComp
 $Comp
-L GND #PWR017
+L GND #PWR29
 U 1 1 57592DA0
 P 7200 1100
-F 0 "#PWR017" H 7200 850 50  0001 C CNN
+F 0 "#PWR29" H 7200 850 50  0001 C CNN
 F 1 "GND" H 7200 950 50  0000 C CNN
 F 2 "" H 7200 1100 50  0000 C CNN
@@
 $EndComp
 $Comp
-L +3V3 #PWR018
+L +3V3 #PWR14
 U 1 1 57599355
 P 3000 4950
-F 0 "#PWR018" H 3000 4800 50  0001 C CNN
+F 0 "#PWR14" H 3000 4800 50  0001 C CNN
 F 1 "+3V3" V 3000 5150 50  0000 C CNN
 F 2 "" H 3000 4950 50  0000 C CNN
@@
 $EndComp
 $Comp
-L GND #PWR019
+L GND #PWR1
 U 1 1 57599CC0
 P 750 7050
-F 0 "#PWR019" H 750 6800 50  0001 C CNN
+F 0 "#PWR1" H 750 6800 50  0001 C CNN
 F 1 "GND" H 750 6900 50  0000 C CNN
 F 2 "" H 750 7050 50  0000 C CNN
@@
 $EndComp
 $Comp
-L GND #PWR020
+L GND #PWR3
 U 1 1 57599E62
 P 1150 6850
-F 0 "#PWR020" H 1150 6600 50  0001 C CNN
+F 0 "#PWR3" H 1150 6600 50  0001 C CNN
 F 1 "GND" H 1150 6700 50  0000 C CNN
 F 2 "" H 1150 6850 50  0000 C CNN
@@
 NoConn ~ 3550 7550
 $Comp
-L GND #PWR021
+L GND #PWR17
 U 1 1 5759B7C2
 P 3150 7550
-F 0 "#PWR021" H 3150 7300 50  0001 C CNN
+F 0 "#PWR17" H 3150 7300 50  0001 C CNN
 F 1 "GND" H 3150 7400 50  0000 C CNN
 F 2 "" H 3150 7550 50  0000 C CNN
@@
 $EndComp
 $Comp
-L +5V #PWR022
+L +5V #PWR2
 U 1 1 5759E11F
 P 1050 4950
-F 0 "#PWR022" H 1050 4800 50  0001 C CNN
+F 0 "#PWR2" H 1050 4800 50  0001 C CNN
 F 1 "+5V" V 1050 5150 50  0000 C CNN
 F 2 "" H 1050 4950 50  0000 C CNN
@@
 $EndComp
 $Comp
-L +3V3 #PWR023
+L +3V3 #PWR22
 U 1 1 5759E6E9
 P 4250 5250
-F 0 "#PWR023" H 4250 5100 50  0001 C CNN
+F 0 "#PWR22" H 4250 5100 50  0001 C CNN
 F 1 "+3V3" H 4250 5390 50  0000 C CNN
 F 2 "" H 4250 5250 50  0000 C CNN
@@
 5V_IN
 $Comp
-L +5V #PWR024
+L +5V #PWR4
 U 1 1 575C79F8
 P 1650 4350
-F 0 "#PWR024" H 1650 4200 50  0001 C CNN
+F 0 "#PWR4" H 1650 4200 50  0001 C CNN
 F 1 "+5V" V 1650 4550 50  0000 C CNN
 F 2 "" H 1650 4350 50  0000 C CNN
@@
 P0.31
 $Comp
-L +3V3 #PWR025
+L +3V3 #PWR16
 U 1 1 575CB207
 P 3150 700
-F 0 "#PWR025" H 3150 550 50  0001 C CNN
+F 0 "#PWR16" H 3150 550 50  0001 C CNN
 F 1 "+3V3" H 3150 850 50  0000 C CNN
 F 2 "" H 3150 700 50  0000 C CNN
@@
 $EndComp
 $Comp
-L GND #PWR026
+L GND #PWR20
 U 1 1 575D0E9A
 P 3650 4500
-F 0 "#PWR026" H 3650 4250 50  0001 C CNN
+F 0 "#PWR20" H 3650 4250 50  0001 C CNN
 F 1 "GND" V 3649 4312 50  0000 C CNN
 F 2 "" H 3650 4500 50  0000 C CNN
@@
 $EndComp
 $Comp
-L GND #PWR027
+L GND #PWR27
 U 1 1 575D0EA0
 P 5200 4500
-F 0 "#PWR027" H 5200 4250 50  0001 C CNN
+F 0 "#PWR27" H 5200 4250 50  0001 C CNN
 F 1 "GND" V 5199 4312 50  0000 C CNN
 F 2 "" H 5200 4500 50  0000 C CNN
@@
 SWDCLK
 $Comp
-L +5V #PWR028
+L +5V #PWR21
 U 1 1 575DB331
 P 4050 5250
-F 0 "#PWR028" H 4050 5100 50  0001 C CNN
+F 0 "#PWR21" H 4050 5100 50  0001 C CNN
 F 1 "+5V" H 4050 5400 50  0000 C CNN
 F 2 "" H 4050 5250 50  0000 C CNN
@@
 $EndComp
 $Comp
-L PWR_FLAG #FLG029
+L PWR_FLAG #FLG1
 U 1 1 575DB491
 P 1600 4250
-F 0 "#FLG029" H 1600 4345 50  0001 C CNN
+F 0 "#FLG1" H 1600 4345 50  0001 C CNN
 F 1 "PWR_FLAG" H 1600 4450 50  0000 C CNN
 F 2 "" H 1600 4250 50  0000 C CNN
@@
 SWO
 $Comp
-L GND #PWR030
+L GND #PWR34
 U 1 1 575DC1F5
 P 9200 4150
-F 0 "#PWR030" H 9200 3900 50  0001 C CNN
+F 0 "#PWR34" H 9200 3900 50  0001 C CNN
 F 1 "GND" V 9200 3950 50  0000 C CNN
 F 2 "" H 9200 4150 50  0000 C CNN
@@
 $EndComp
 $Comp
-L +3V3 #PWR031
+L +3V3 #PWR35
 U 1 1 575DC6AD
 P 9200 4250
-F 0 "#PWR031" H 9200 4100 50  0001 C CNN
+F 0 "#PWR35" H 9200 4100 50  0001 C CNN
 F 1 "+3V3" V 9201 4478 50  0000 C CNN
 F 2 "" H 9200 4250 50  0000 C CNN
@@
 $EndComp
 $Comp
-L GND #PWR032
+L GND #PWR33
 U 1 1 575DC996
 P 8450 5850
-F 0 "#PWR032" H 8450 5600 50  0001 C CNN
+F 0 "#PWR33" H 8450 5600 50  0001 C CNN
 F 1 "GND" V 8450 5650 50  0000 C CNN
 F 2 "" H 8450 5850 50  0000 C CNN
@@
 $EndComp
 $Comp
-L +3V3 #PWR033
+L +3V3 #PWR31
 U 1 1 575DCAE2
 P 8450 5550
-F 0 "#PWR033" H 8450 5400 50  0001 C CNN
+F 0 "#PWR31" H 8450 5400 50  0001 C CNN
 F 1 "+3V3" V 8449 5773 50  0000 C CNN
 F 2 "" H 8450 5550 50  0000 C CNN
@@
 $EndComp
 $Comp
-L GND #PWR034
+L GND #PWR32
 U 1 1 575DCBF4
 P 8450 5650
-F 0 "#PWR034" H 8450 5400 50  0001 C CNN
+F 0 "#PWR32" H 8450 5400 50  0001 C CNN
 F 1 "GND" V 8450 5450 50  0000 C CNN
 F 2 "" H 8450 5650 50  0000 C CNN
@@
 $EndComp
 $Comp
-L +3V3 #PWR035
+L +3V3 #PWR6
 U 1 1 575DCF2A
 P 2050 6350
-F 0 "#PWR035" H 2050 6200 50  0001 C CNN
+F 0 "#PWR6" H 2050 6200 50  0001 C CNN
 F 1 "+3V3" V 2050 6600 50  0000 C CNN
 F 2 "" H 2050 6350 50  0000 C CNN
@@
 $EndComp
 $Comp
-L GND #PWR036
+L GND #PWR24
 U 1 1 575DD677
 P 4650 5600
-F 0 "#PWR036" H 4650 5350 50  0001 C CNN
+F 0 "#PWR24" H 4650 5350 50  0001 C CNN
 F 1 "GND" H 4650 5450 50  0000 C CNN
 F 2 "" H 4650 5600 50  0000 C CNN
@@
 $EndComp
 $Comp
-L GND #PWR037
+L GND #PWR23
 U 1 1 575DED7D
 P 4650 5350
-F 0 "#PWR037" H 4650 5100 50  0001 C CNN
+F 0 "#PWR23" H 4650 5100 50  0001 C CNN
 F 1 "GND" H 4650 5200 50  0000 C CNN
 F 2 "" H 4650 5350 50  0000 C CNN
@@
 	4250 5250 4250 5650
 $Comp
-L CONN_01X01 P?
-U 1 1 5762FAFE
-P 8650 1650
-F 0 "P?" H 8728 1691 50  0000 L CNN
-F 1 "CONN_01X01" H 8728 1600 50  0000 L CNN
-F 2 "" H 8650 1650 50  0000 C CNN
-F 3 "" H 8650 1650 50  0000 C CNN
-	1    8650 1650
-	1    0    0    -1
-$EndComp
+L CONN_02X01 P4
+U 1 1 57630A50
+P 8000 1150
+F 0 "P4" H 8000 925 50  0000 C CNN
+F 1 "ANTENNA_2_4GHZ" H 8000 1016 50  0000 C CNN
+F 2 "xil_assets:ti-an043-antenna" H 8000 -50 50  0001 C CNN
+F 3 "" H 8000 -50 50  0000 C CNN
+	1    8000 1150
+	1    0    0    1
+$EndComp
+Wire Wire Line
+	7750 1150 7750 800
+Connection ~ 7750 800
+$Comp
+L GND #PWR30
+U 1 1 57630CDC
+P 8250 1150
+F 0 "#PWR30" H 8250 900 50  0001 C CNN
+F 1 "GND" H 8250 1000 50  0000 C CNN
+F 2 "" H 8250 1150 50  0000 C CNN
+F 3 "" H 8250 1150 50  0000 C CNN
+	1    8250 1150
+	1    0    0    -1
+$EndComp

Commit message: WIP IT! Finally somethings nice yo.
Parts:
- removed D1, D2: D, Diodes_SMD:DO-214BA, symbol D
- added D1, D2: D_Schottky, Diodes_SMD:SOD-123, symbol D_Schottky
Connections:
- net +3V3: now also D2.1 (K)
- net +5V: now also D1.1 (K)
- net 5V_IN: now also D1.2 (A)
- net at U3.3 (OUT): now also D2.2 (A)

Commit message: Make it nicer
Changed lines of the file:
@@
 LIBS:tmp007
 LIBS:uvis25
-LIBS:tom_kicad
 LIBS:nrf52_rev1-cache
 EELAYER 25 0
@@
 Text GLabel 9550 4850 2    47   Input ~ 0
 RESET
-Text GLabel 9600 5150 2    47   Input ~ 0
+Text GLabel 9550 5150 2    47   Input ~ 0
 SWO
 $Comp
