File: rev_a1/CP2102.sch (KiCad schematic (older format))
At the start: 5 parts, among them P3 USB_OTG, U2 CP2102

Commit message: final touches
Connections:
- net +5V is gone; now on net USB_VBUS: U2.8 (VBUS)
Changed lines of the file:
@@
 $EndComp
 $Comp
-L GND #PWR035
+L GND #PWR32
 U 1 1 5765BA43
 P 3300 4100
-F 0 "#PWR035" H 3300 3850 50  0001 C CNN
+F 0 "#PWR32" H 3300 3850 50  0001 C CNN
 F 1 "GND" H 3300 3950 50  0000 C CNN
 F 2 "" H 3300 4100 50  0000 C CNN
@@
 $EndComp
 $Comp
-L GND #PWR036
+L GND #PWR33
 U 1 1 5765BA49
 P 3700 3900
-F 0 "#PWR036" H 3700 3650 50  0001 C CNN
+F 0 "#PWR33" H 3700 3650 50  0001 C CNN
 F 1 "GND" H 3700 3750 50  0000 C CNN
 F 2 "" H 3700 3900 50  0000 C CNN
@@
 NoConn ~ 6100 4600
 $Comp
-L GND #PWR037
+L GND #PWR35
 U 1 1 5765BA62
 P 5700 4600
-F 0 "#PWR037" H 5700 4350 50  0001 C CNN
+F 0 "#PWR35" H 5700 4350 50  0001 C CNN
 F 1 "GND" H 5700 4450 50  0000 C CNN
 F 2 "" H 5700 4600 50  0000 C CNN
@@
 Configured to bypass internal regulator.\nUses our 5v to 3v3 regulator.
 $Comp
-L +3V3 #PWR038
+L +3V3 #PWR36
 U 1 1 5765BA6F
 P 6800 2300
-F 0 "#PWR038" H 6800 2150 50  0001 C CNN
+F 0 "#PWR36" H 6800 2150 50  0001 C CNN
 F 1 "+3V3" H 6800 2440 50  0000 C CNN
 F 2 "" H 6800 2300 50  0000 C CNN
@@
 	1    6800 2300
 	1    0    0    -1
-$EndComp
-$Comp
-L +5V #PWR039
-U 1 1 5765BA7D
-P 6600 2300
-F 0 "#PWR039" H 6600 2150 50  0001 C CNN
-F 1 "+5V" H 6600 2450 50  0000 C CNN
-F 2 "" H 6600 2300 50  0000 C CNN
-F 3 "" H 6600 2300 50  0000 C CNN
-	1    6600 2300
-	-1   0    0    -1
 $EndComp
 $Comp
@@
 $EndComp
 $Comp
-L +3V3 #PWR040
+L +3V3 #PWR34
 U 1 1 5765BA8D
 P 4600 3400
-F 0 "#PWR040" H 4600 3250 50  0001 C CNN
+F 0 "#PWR34" H 4600 3250 50  0001 C CNN
 F 1 "+3V3" V 4600 3650 50  0000 C CNN
 F 2 "" H 4600 3400 50  0000 C CNN
@@
 $EndComp
 $Comp
-L GND #PWR041
+L GND #PWR38
 U 1 1 5765BA9A
 P 7200 2650
-F 0 "#PWR041" H 7200 2400 50  0001 C CNN
+F 0 "#PWR38" H 7200 2400 50  0001 C CNN
 F 1 "GND" H 7200 2500 50  0000 C CNN
 F 2 "" H 7200 2650 50  0000 C CNN
@@
 $EndComp
 $Comp
-L GND #PWR042
+L GND #PWR37
 U 1 1 5765BAA0
 P 7200 2400
-F 0 "#PWR042" H 7200 2150 50  0001 C CNN
+F 0 "#PWR37" H 7200 2150 50  0001 C CNN
 F 1 "GND" H 7200 2250 50  0000 C CNN
 F 2 "" H 7200 2400 50  0000 C CNN
@@
 Text HLabel 3700 3500 2    47   Output ~ 0
 USB_VBUS
+Text HLabel 6600 2300 1    47   Output ~ 0
+USB_VBUS
 $EndSCHEMATC
